File: hardware/brain-board/pcb/brain.brd (EAGLE design)
At the start: 46.5 x 40.3 mm, 17 parts, among them Y2 16MHz

Commit message: Brain Rev B
Parts:
- removed ATMEGA328: ATMEGA328P-20MU, idii:MLF32
- removed C6: 100n, SmartPrj:C0603-ROUND
- removed I2CIN, I2COUT, LED1: (no value), SparkFun:1X04_LONGPADS
- removed ICSP: ICSP, pinhead:2X03
- removed MOTOR1, MOTOR2, MOTOR3: (no value), SparkFun:1X03
- removed R1, R2: 10K, resistor:R0603
- removed R5, R6, R7: 470, resistor:R0603
- removed Y2: 16MHz, SmartPrj:RESONATOR
- added ADC6, ADC7, AGND, AREF, CTS, GND, PD2, PD4, PD7, RTS: TEST_POINT_SM_2X2, test-points:TP-SMT-020X020
- added ADDR: CTS_219-04MST, switch-smd:CTS_4P_GULLWING
- added C1, C2: 0.1uF, rlc:0603
- added CR1: (no value), ceramic-resonators:MURATA_CSTCE
- added I2CA, I2CB: (no value), con-headers:MA04-1-RA
- added ISCP: (no value), con-headers:MA03-2
- added J5: (no value), con-headers:MA06-1-EDGE-2.54MM
- added LEDS: (no value), con-headers:MA04-1
- added LOGO1: SPETKU-14MM, logos:SPETKU_14MM
- added LOGO2: LIGHT_PLAY_20MM, logos:LIGHTPLAY_20MM
- added Q1: SI2302CDS, transistor-fet:SOT-23
- added R10, R9: NS, rlc:0603
- added R11, R12, R13: 470, rlc:0603
- added R16: CTS 741X163102JP, rlc:RESNET_0402_X8
- added R8: 10K, rlc:0603
- added RESET: (no value), switch-smd:B3FS
- added SV1, SV2, SV3: (no value), con-headers:MA03-1
- added U1: ATmega328P-AU, atmel-atmega:TQFP-32-08
- R3: value 10K -> NS; device resistor:R0603 -> rlc:0603
- R4: value 1M -> 100K; device resistor:R0603 -> rlc:0603
- moved R3 92.1 mm to (8.60, -12.0), turned to 0 degrees
- moved R4 91.9 mm to (-11.1, -9.00), turned to 0 degrees
Connections:
- removed net +5V: ATMEGA328.18, ATMEGA328.4, ATMEGA328.6, C6.2, I2CIN.1, I2COUT.1, ICSP.2, MOTOR1.2, MOTOR2.2, MOTOR3.2, R1.2, R2.2, R3.2
- removed net N$13: ATMEGA328.1, R5.2
- new net AREF: AREF.1, U1.20
- new net CTS: CTS.1, J5.2
- new net D3: R13.1, U1.1
- new net D5: R12.1, U1.9
- new net D6: R11.1, U1.10
- new net LED_B: LEDS.1, R11.2
- new net LED_G: LEDS.2, R12.2
- new net LED_R: LEDS.3, R13.2
- new net N$19: R16.6, U1.14
- new net N$2: Q1.3, SV1.3, SV2.3, SV3.3
- new net N$20: R16.7, U1.13
- new net N$21: ADDR.2, U1.25
- new net N$22: ADDR.3, U1.24
- new net N$23: ADDR.4, U1.23
- new net N$4: ADDR.1, U1.26
- new net N$5: R16.10, SV3.1
- new net RTS: C2.2, J5.6, RTS.1
- new net RX: R16.3, U1.30
- new net RXD: J5.5, R16.13
- new net SCL: I2CA.1, I2CB.1, R16.15, R9.1
- new net SDA: I2CA.2, I2CB.2, R10.1, R16.16
- new net SERVO_EN: Q1.1, R4.2, U1.12
- new net TX: R16.4, U1.31
- new net TXD: J5.4, R16.14
- new net VCC: C1.1, I2CA.3, I2CB.3, ISCP.2, R10.2, R3.1, R8.2, R9.2, SV1.2, SV2.2, SV3.2, U1.18, U1.4, U1.6
- new net VCC5: J5.3, R3.2
- net GND: now also ADDR.5, ADDR.6, ADDR.7, ADDR.8, AGND.1, C1.2, CR1.2, GND.1, I2CA.4, I2CB.4, ISCP.6, J5.1, LEDS.4, Q1.2, R4.1, RESET.3, RESET.4, U1.21, U1.3, U1.5; no longer ATMEGA328.21, ATMEGA328.3, ATMEGA328.5, C6.1, I2CIN.4, I2COUT.4, ICSP.6, LED1.4, MOTOR1.3, MOTOR2.3, MOTOR3.3, Y2.2
- net MISO: now also ISCP.1, U1.16; no longer ATMEGA328.16, ICSP.1
- net MOSI: now also ISCP.4, R16.5, U1.15; no longer ATMEGA328.15, ICSP.4, MOTOR1.1
- net N$1: now also PD2.1, U1.32; no longer ATMEGA328.28, I2CIN.2, I2COUT.2, R2.1
- net N$10: now also R16.12, SV1.1; no longer ATMEGA328.13, MOTOR3.1
- net N$11: now also R16.2, U1.28; no longer ATMEGA328.10, R7.2
- net N$12: now also R16.1, U1.27; no longer ATMEGA328.9, R6.2
- net N$3: now also PD4.1, U1.2; no longer ATMEGA328.27, I2CIN.3, I2COUT.3, R3.1
- net N$6: now also PD7.1, U1.11; no longer LED1.1, R7.1
- net N$7: now also ADC6.1, U1.19; no longer LED1.2, R6.1
- net N$8: now also ADC7.1, U1.22; no longer LED1.3, R5.1
- net N$9: now also R16.11, SV2.1; no longer ATMEGA328.14, MOTOR2.1
- net RESET: now also C2.1, ISCP.5, R8.1, RESET.1, RESET.2, U1.29; no longer ATMEGA328.29, ICSP.5, R1.1
- net SCK: now also ISCP.3, U1.17; no longer ATMEGA328.17, ICSP.3
- net XTAL1: now also CR1.3, U1.7; no longer ATMEGA328.7, R4.1, Y2.3
- net XTAL2: now also CR1.1, U1.8; no longer ATMEGA328.8, R4.2, Y2.1
Routing:
- net +5V: track 117.3 -> 0.00 mm, vias 3 -> 0
- net VCC: track 0.00 -> 117.3 mm, vias 0 -> 2
- net RESET: track 17.3 -> 96.3 mm, vias 1 -> 4
- net SCL: track 0.00 -> 60.3 mm
- net SDA: track 0.00 -> 59.6 mm
- net N$13: track 29.7 -> 0.00 mm
- net N$3: track 46.7 -> 18.2 mm, vias 0 -> 1
- net AREF: track 0.00 -> 28.5 mm, vias 0 -> 1
- net N$1: track 45.1 -> 17.9 mm, vias 0 -> 1
- net D3: track 0.00 -> 26.5 mm, vias 0 -> 4
- net N$7: track 2.93 -> 26.3 mm, vias 0 -> 1
- net D6: track 0.00 -> 22.8 mm
- net N$6: track 2.94 -> 23.4 mm, vias 0 -> 1
- net N$8: track 2.94 -> 22.3 mm, vias 0 -> 1
- net D5: track 0.00 -> 18.1 mm
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Other:
- board size 46.5 x 40.3 mm -> 50 x 43.3 mm
- board text added: "+"
- board text added: "G"
- board text added: "LIGHTPLAY.ZONESS.COM 2013"
- board text added: "Light"
- board text added: "Light Play"
- board text added: "Play"
- board text added: "Rev. B"
- board text added: "S"
- board text removed: "DELTA DELTA DELTA"
- board text removed: "KRUX<3"
- board text removed: "Z1"
- board text removed: "ZONESS.COM 2013"
- board text removed: "circuitMonkey"

Commit message: rev-c board
Parts:
- removed I2CA, I2CB: (no value), con-headers:MA04-1-RA
- removed J5: (no value), con-headers:MA06-1-EDGE-2.54MM
- removed LOGO1: SPETKU-14MM, logos:SPETKU_14MM
- added C3: 0.01uF, rlc:0603
- added C5: 10uF, rlc:0805
- added C6: 0.1uF, rlc:0603
- added C7: 220uF/6.3V, rlc:CAP_ALUM_SMT_6.3
- added D1: Toshiba 1SS416CT, diodes:CST2
- added I/O: (no value), con-headers:MA04-1
- added JMP1: (no value), con-headers:MA02-1-FAT
- added SERIAL: (no value), con-headers:MA06-1
- CR1: value (none) -> Murata CSTCE 16Mhz
- R11, R12, R13: value 470 -> 220
- R4: value 100K -> 160K
- RESET: value (none) -> B3FS
- moved Q1 2.74 mm to (-7.00, -12.7)
- moved CR1 1.60 mm to (-7.80, -2.51)
- moved ISCP 1.57 mm to (14.4, 7.76)
- moved RESET 0.11 mm to (-15.0, 10.4)
Connections:
- new net N$13: C2.1, JMP1.2
- new net VCC_AVR: C1.1, C3.1, C7.+, D1.K, R8.2, U1.18, U1.4, U1.6
- net CTS: now also SERIAL.2; no longer J5.2
- net GND: now also C3.2, C5.2, C6.2, C7.-, I/O.4, SERIAL.1; no longer I2CA.4, I2CB.4, J5.1
- net RESET: now also C5.1, JMP1.1; no longer C2.1
- net RTS: now also SERIAL.6; no longer J5.6
- net RXD: now also SERIAL.5; no longer J5.5
- net SCL: now also I/O.1; no longer I2CA.1, I2CB.1
- net SDA: now also I/O.2; no longer I2CA.2, I2CB.2
- net TXD: now also SERIAL.4; no longer J5.4
- net VCC: now also C6.1, D1.A, I/O.3; no longer C1.1, I2CA.3, I2CB.3, R8.2, U1.18, U1.4, U1.6
- net VCC5: now also SERIAL.3; no longer J5.3
Routing:
- net RESET: track 96.3 -> 57.1 mm, vias 4 -> 2
- net VCC: track 117.3 -> 78.1 mm
- net VCC_AVR: track 0.00 -> 34.2 mm
- net N$13: track 0.00 -> 22.9 mm
- net CTS: track 13.4 -> 9.28 mm
- net SDA: track 59.6 -> 55.6 mm, vias 0 -> 1
- net SCL: track 60.3 -> 57.0 mm, vias 0 -> 1
- net SERVO_EN: track 14.6 -> 17.4 mm
- net VCC5: track 14.4 -> 12.2 mm, vias 1 -> 0
- net XTAL2: track 5.48 -> 3.84 mm
- net XTAL1: track 5.39 -> 3.75 mm
- net N$2: track 11.2 -> 9.70 mm
- net TXD: track 11.4 -> 10.1 mm
- net RXD: track 11.6 -> 10.5 mm
- net D3: track 26.5 -> 27.6 mm
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Other:
- board text added: "<3"
- board text added: "Command & Cuddle"
- board text added: "Petkus | Koch"
- board text added: "R O B O T - A R M Y . C O M"
- board text added: "ROBOT-ARMY.COM 2013"
- board text added: "Rev. C"
- board text added: "Robot Army"
- board text removed: "LIGHTPLAY.ZONESS.COM 2013"
- board text removed: "Light"
- board text removed: "Light Play"
- board text removed: "Play"
- board text removed: "Rev. B"

Commit message: rev-d board
Parts:
- removed C7: 220uF/6.3V, rlc:CAP_ALUM_SMT_6.3
- removed D1: Toshiba 1SS416CT, diodes:CST2
- removed R13: 220, rlc:0603
- removed R16: CTS 741X163102JP, rlc:RESNET_0402_X8
- added C4: 0.01uF, rlc:0603
- added R1, R2: 10K, rlc:0603
- C3: value 0.01uF -> 0.1uF
- C6: value 0.1uF -> 220uF/6.3V; device rlc:0603 -> rlc:CAP_ALUM_SMT_6.3
- Q1: value SI2302CDS -> 2N7002
- R4: value 160K -> NS
- R8: value 10K -> 220
- R9: value NS -> CTS 741X163102JP; device rlc:0603 -> rlc:RESNET_0402_X8
- moved R4 19.7 mm to (8.60, -9.30), turned to 180 degrees
- moved R8 16.5 mm to (-11.1, -10.4)
- moved C3 14.6 mm to (-6.93, -12.9)
- moved C6 11.1 mm to (-14.6, -1.07), turned to 120 degrees
- moved R9 6.55 mm to (9.40, -2.80), turned to 0 degrees
- moved Q1 2.76 mm to (-6.93, -9.98)
- moved ISCP 1.06 mm to (14.1, 8.77), turned to 300 degrees
- renumbered R10 to R5, R11 to R6, R12 to R7
Connections:
- removed net VCC_AVR: C1.1, C3.1, C7.+, D1.K, R8.2, U1.18, U1.4, U1.6
- net D3: now also R8.1; no longer R13.1
- net GND: now also C4.2, C6.-, SV1.3, SV2.3, SV3.3; no longer C6.2, C7.-, R4.1
- net LED_R: now also R8.2; no longer R13.2
- net MOSI: now also R9.5; no longer R16.5
- net N$10: now also Q1.3, R9.11, R9.12; no longer R16.12, SV1.1
- net N$11: now also R9.2; no longer R16.2
- net N$12: now also R9.1; no longer R16.1
- net N$19: now also R9.7; no longer R16.6
- net N$2: now also R9.6, SV1.1; no longer Q1.3, SV1.3, SV2.3, SV3.3
- net N$20: now also R9.8; no longer R16.7
- net N$5: now also R9.9; no longer R16.10
- net N$9: now also R9.10; no longer R16.11
- net RESET: now also R1.1; no longer R8.1
- net RX: now also R9.3; no longer R16.3
- net RXD: now also R9.13; no longer R16.13
- net SCL: now also R4.1, R9.15; no longer R16.15, R9.1
- net SDA: now also R9.16; no longer R16.16
- net SERVO_EN: now also R2.2; no longer R4.2
- net TX: now also R9.4; no longer R16.4
- net TXD: now also R9.14; no longer R16.14
- net VCC: now also C1.1, C3.1, C4.1, C6.+, R1.2, R2.1, R4.2, U1.18, U1.4, U1.6; no longer C6.1, D1.A, R9.2
Routing:
- net VCC: track 78.1 -> 118.0 mm, vias 2 -> 3
- net VCC_AVR: track 34.2 -> 0.00 mm
- net N$10: track 14.8 -> 25.0 mm
- net RESET: track 57.1 -> 47.9 mm, vias 2 -> 3
- net N$2: track 9.70 -> 17.2 mm, vias 0 -> 2
- net MOSI: track 24.8 -> 30.0 mm, vias 2 -> 1
- net SCK: track 21.7 -> 16.6 mm, vias 2 -> 0
- net SERVO_EN: track 17.4 -> 14.3 mm
- net N$5: track 17.9 -> 15.1 mm
- net N$9: track 16.4 -> 14.1 mm
- net N$19: track 11.1 -> 9.85 mm
- net N$20: track 11.9 -> 10.8 mm
- net MISO: track 20.9 -> 20.0 mm
- net D3: track 27.6 -> 26.7 mm
Other:
- board text added: "ROBOT ARMY"
- board text added: "ROBOT-ARMY.COM 2014"
- board text added: "Rev. D"
- board text removed: "ROBOT-ARMY.COM 2013"
- board text removed: "Rev. C"
- board text removed: "Robot Army"

Commit message: rev-e board
Parts:
- removed I/O: (no value), con-headers:MA04-1
- removed JMP1: (no value), con-headers:MA02-1-FAT
- removed PD2, PD4, PD7: TEST_POINT_SM_2X2, test-points:TP-SMT-020X020
- removed R4, R5: NS, rlc:0603
- removed R6, R7, R8: 220, rlc:0603
- removed R9: CTS 741X163102JP, rlc:RESNET_0402_X8
- added AIN4, AIN5, D2, D4, D7: TEST_POINT_SM_2X2, test-points:TP-SMT-020X020
- added D1: Toshiba 1SS416CT, diodes:CST2
- added D13: YEL, led:SMD_0603
- added POWER: HDR, M, 3P, con-headers:MA03-1
- added SER_PWR, SER_RST: (no value), con-headers:MA02-1-FAT
- C6: value 220uF/6.3V -> 1000uF/10V; device rlc:CAP_ALUM_SMT_6.3 -> rlc:CAP_ALUM_THD_8
- R3: value NS -> CTS 741X163102JP; device rlc:0603 -> rlc:RESNET_0402_X8
- moved GND 12.3 mm to (-21.1, 3.81)
- moved R3 9.23 mm to (9.40, -2.80)
- moved R2 4.68 mm to (-6.93, -6.87)
- moved C6 3.21 mm to (-17.6, 0.15), turned to 180 degrees
- moved Q1 0.08 mm to (-6.93, -9.91)
Connections:
- removed net D3: R8.1, U1.1
- removed net D5: R7.1, U1.9
- removed net D6: R6.1, U1.10
- removed net SCL: I/O.1, R4.1, R9.15
- removed net SDA: I/O.2, R5.1, R9.16
- new net N$17: D13.A, R3.16
- new net PWR_IN: C3.1, D1.A, ISCP.2, LEDS.4, POWER.2, SER_PWR.1, SV1.2, SV2.2, SV3.2
- net GND: now also C6.N, D13.K, POWER.3; no longer C6.-, I/O.4, LEDS.4
- net LED_B: now also U1.10; no longer R6.2
- net LED_G: now also U1.9; no longer R7.2
- net LED_R: now also U1.1; no longer R8.2
- net MOSI: now also R3.5; no longer R9.5
- net N$1: now also D2.1; no longer PD2.1
- net N$10: now also R3.11, R3.12; no longer R9.11, R9.12
- net N$11: now also AIN5.1; no longer R9.2
- net N$12: now also AIN4.1; no longer R9.1
- net N$13: now also SER_RST.2; no longer JMP1.2
- net N$19: now also R3.7; no longer R9.7
- net N$2: now also R3.6; no longer R9.6
- net N$20: now also R3.8; no longer R9.8
- net N$3: now also D4.1; no longer PD4.1
- net N$5: now also R3.9; no longer R9.9
- net N$6: now also D7.1; no longer PD7.1
- net N$9: now also R3.10; no longer R9.10
- net RESET: now also POWER.1, SER_RST.1; no longer JMP1.1
- net RX: now also R3.3; no longer R9.3
- net RXD: now also R3.13; no longer R9.13
- net SCK: now also R3.1
- net TX: now also R3.4; no longer R9.4
- net TXD: now also R3.14; no longer R9.14
- net VCC: now also C6.P, D1.K; no longer C3.1, C6.+, I/O.3, ISCP.2, R3.1, R4.2, R5.2, SV1.2, SV2.2, SV3.2
- net VCC5: now also SER_PWR.2; no longer R3.2
Routing:
- net PWR_IN: track 0.00 -> 73.1 mm
- net VCC: track 118.0 -> 47.4 mm, vias 3 -> 2
- net SCL: track 57.0 -> 0.00 mm, vias 1 -> 0
- net SDA: track 55.4 -> 0.00 mm, vias 1 -> 0
- net D3: track 26.7 -> 0.00 mm, vias 4 -> 0
- net RESET: track 47.9 -> 74.2 mm
- net LED_R: track 15.4 -> 40.7 mm, vias 0 -> 4
- net D6: track 23.3 -> 0.00 mm
- net D5: track 18.7 -> 0.00 mm
- net LED_G: track 11.4 -> 25.5 mm
- net LED_B: track 8.04 -> 21.8 mm
- net N$12: track 12.9 -> 20.9 mm, vias 2 -> 1
- net SCK: track 16.6 -> 22.3 mm
- net N$11: track 14.8 -> 20.0 mm, vias 2 -> 1
- net SERVO_EN: track 14.3 -> 9.41 mm
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Other:
- board text added: "&"
- board text added: "Command"
- board text added: "Cuddle"
- board text added: "GND"
- board text added: "RESET"
- board text added: "Rev. E"
- board text removed: "Command & Cuddle"
- board text removed: "Rev. D"
