File: hardware/brain-board/pcb/brain.sch (EAGLE design)
At the start: 17 parts, among them Y2 16MHz

Commit message: Brain Rev B
Parts:
- removed ATMEGA328: ATMEGA328P-20MU, idii:MEGA8-MI
- removed C6: 100n, SmartPrj:C-EU0603-RND
- removed I2CIN, I2COUT, LED1: (no value), SparkFun:M04LONGPADS
- removed ICSP: ICSP, pinhead:PINHD-2X3
- removed MOTOR1, MOTOR2, MOTOR3: (no value), SparkFun:M03PTH
- removed R1, R2: 10K, resistor:R-US_R0603
- removed R5, R6, R7: 470, resistor:R-US_R0603
- removed Y2: 16MHz, SmartPrj:RESONATORMU
- added ADC6, ADC7, AGND, AREF, CTS, GND, PD2, PD4, PD7, RTS: TEST_POINT_SM_2X2, test-points:TEST_POINT_SM_2X2
- added ADDR: CTS_219-04MST, switch-smd:DIP-4PCTS-219-SMD
- added C1, C2: 0.1uF, rlc:CAPACITOR0603
- added CR1: (no value), ceramic-resonators:RESONATORMURATA-CSTCE
- added I2CA, I2CB: (no value), con-headers:MA04-1-RA
- added ISCP: (no value), con-headers:MA03-2
- added J5: (no value), con-headers:MA06-1-EDGE
- added LEDS: (no value), con-headers:MA04-1
- added LOGO1: SPETKU-14MM, logos:SPETKU-14MM
- added LOGO2: LIGHT_PLAY_20MM, logos:LIGHT_PLAY_20MM
- added Q1: SI2302CDS, transistor-fet:SOT23_SI2302
- added R10, R9: NS, rlc:RESISTOR0603
- added R11, R12, R13: 470, rlc:RESISTOR0603
- added R16: CTS 741X163102JP, rlc:RESNET_0402_INDIV_X8
- added R8: 10K, rlc:RESISTOR0603
- added RESET: (no value), switch-smd:PUSHBTN-SP-MOM-4PINB3FS
- added SV1, SV2, SV3: (no value), con-headers:MA03-1
- added U1: ATmega328P-AU, atmel-atmega:ATMEGA328
- R3: value 10K -> NS; device resistor:R-US_R0603 -> rlc:RESISTOR0603
- R4: value 1M -> 100K; device resistor:R-US_R0603 -> rlc:RESISTOR0603
Connections:
- removed net +5V: ATMEGA328.AVCC, ATMEGA328.VCC@1, ATMEGA328.VCC@2, C6.2, I2CIN.1, I2COUT.1, ICSP.2, MOTOR1.2, MOTOR2.2, MOTOR3.2, R1.2, R2.2, R3.2
- removed net N$13: ATMEGA328.PD3(INT1), R5.2
- new net AREF: AREF.P$1, U1.AREF
- new net CTS: CTS.P$1, J5.2
- new net D3: R13.1, U1.PD3
- new net D5: R12.1, U1.PD5
- new net D6: R11.1, U1.PD6
- new net LED_B: LEDS.1, R11.2
- new net LED_G: LEDS.2, R12.2
- new net LED_R: LEDS.3, R13.2
- new net N$19: R16F.1, U1.PB2
- new net N$2: Q1.D, SV1.3, SV2.3, SV3.3
- new net N$20: R16G.1, U1.PB1
- new net N$21: ADDR.2, U1.PC2
- new net N$22: ADDR.3, U1.PC1
- new net N$23: ADDR.4, U1.PC0
- new net N$4: ADDR.1, U1.PC3
- new net N$5: R16G.2, SV3.1
- new net RTS: C2.2, J5.6, RTS.P$1
- new net RX: R16C.1, U1.PD0
- new net RXD: J5.5, R16D.2
- new net SCL: I2CA.1, I2CB.1, R16B.2, R9.1
- new net SDA: I2CA.2, I2CB.2, R10.1, R16A.2
- new net SERVO_EN: Q1.G, R4.2, U1.PB0
- new net TX: R16D.1, U1.PD1
- new net TXD: J5.4, R16C.2
- new net VCC: C1.1, I2CA.3, I2CB.3, ISCP.2, R10.2, R3.1, R8.2, R9.2, SV1.2, SV2.2, SV3.2, U1.AVCC, U1.VCC@4, U1.VCC@6
- new net VCC5: J5.3, R3.2
- net GND: now also ADDR.5, ADDR.6, ADDR.7, ADDR.8, AGND.P$1, C1.2, CR1.2, GND.P$1, I2CA.4, I2CB.4, ISCP.6, J5.1, LEDS.4, Q1.S, R4.1, RESET.3, RESET.4, U1.AGND, U1.GND@3, U1.GND@5; no longer ATMEGA328.AGND, ATMEGA328.GND@1, ATMEGA328.GND@2, C6.1, I2CIN.4, I2COUT.4, ICSP.6, LED1.4, MOTOR1.3, MOTOR2.3, MOTOR3.3, Y2.2
- net MISO: now also ISCP.1, U1.PB4; no longer ATMEGA328.PB4(MISO), ICSP.1
- net MOSI: now also ISCP.4, R16E.1, U1.PB3; no longer ATMEGA328.PB3(MOSI/OC2), ICSP.4, MOTOR1.1
- net N$1: now also PD2.P$1, U1.PD2; no longer ATMEGA328.PC5(ADC5/SCL), I2CIN.2, I2COUT.2, R2.1
- net N$10: now also R16E.2, SV1.1; no longer ATMEGA328.PB1(OC1A), MOTOR3.1
- net N$11: now also R16B.1, U1.PC5; no longer ATMEGA328.PD6(AIN0), R7.2
- net N$12: now also R16A.1, U1.PC4; no longer ATMEGA328.PD5(T1), R6.2
- net N$3: now also PD4.P$1, U1.PD4; no longer ATMEGA328.PC4(ADC4/SDA), I2CIN.3, I2COUT.3, R3.1
- net N$6: now also PD7.P$1, U1.PD7; no longer LED1.1, R7.1
- net N$7: now also ADC6.P$1, U1.ADC6; no longer LED1.2, R6.1
- net N$8: now also ADC7.P$1, U1.ADC7; no longer LED1.3, R5.1
- net N$9: now also R16F.2, SV2.1; no longer ATMEGA328.PB2(SS/OC1B), MOTOR2.1
- net RESET: now also C2.1, ISCP.5, R8.1, RESET.1, RESET.2, U1.PC6; no longer ATMEGA328.PC6(/RESET), ICSP.5, R1.1
- net SCK: now also ISCP.3, U1.PB5; no longer ATMEGA328.PB5(SCK), ICSP.3
- net XTAL1: now also CR1.3, U1.PB6; no longer ATMEGA328.PB6(XTAL1/TOSC1), R4.1, Y2.3
- net XTAL2: now also CR1.1, U1.PB7; no longer ATMEGA328.PB7(XTAL2/TOSC2), R4.2, Y2.1
Other:
- note added: "Change to cheaper switch"
- note added: "FTDI-USB-Serial"
- note added: "I2C pull-ups: No stuff for slaves. You only need one set at the master."

Commit message: rev-c board
Parts:
- removed I2CA, I2CB: (no value), con-headers:MA04-1-RA
- removed J5: (no value), con-headers:MA06-1-EDGE
- removed LOGO1: SPETKU-14MM, logos:SPETKU-14MM
- added C3: 0.01uF, rlc:CAPACITOR0603
- added C5: 10uF, rlc:CAPACITOR0805
- added C6: 0.1uF, rlc:CAPACITOR0603
- added C7: 220uF/6.3V, rlc:CAPACITOR_POL-ALUM-SMT-6.3
- added D1: Toshiba 1SS416CT, diodes:SCHOTTKYTOSHIBA_CST2
- added I/O: (no value), con-headers:MA04-1
- added JMP1: (no value), con-headers:JMP01VT
- added SERIAL: (no value), con-headers:MA06-1
- CR1: value (none) -> Murata CSTCE 16Mhz
- R11, R12, R13: value 470 -> 220
- R4: value 100K -> 160K
- RESET: value (none) -> B3FS
Connections:
- new net N$13: C2.1, JMP1.P$2
- new net VCC_AVR: C1.1, C3.1, C7.P, D1.K, R8.2, U1.AVCC, U1.VCC@4, U1.VCC@6
- net CTS: now also SERIAL.2; no longer J5.2
- net GND: now also C3.2, C5.2, C6.2, C7.N, I/O.4, SERIAL.1; no longer I2CA.4, I2CB.4, J5.1
- net RESET: now also C5.1, JMP1.P$1; no longer C2.1
- net RTS: now also SERIAL.6; no longer J5.6
- net RXD: now also SERIAL.5; no longer J5.5
- net SCL: now also I/O.1; no longer I2CA.1, I2CB.1
- net SDA: now also I/O.2; no longer I2CA.2, I2CB.2
- net TXD: now also SERIAL.4; no longer J5.4
- net VCC: now also C6.1, D1.A, I/O.3; no longer C1.1, I2CA.3, I2CB.3, R8.2, U1.AVCC, U1.VCC@4, U1.VCC@6
- net VCC5: now also SERIAL.3; no longer J5.3
Other:
- note added: "470uf"
- note removed: "Change to cheaper switch"
- moved on the sheet: C1, R8, RESET

Commit message: rev-d board
Parts:
- removed C7: 220uF/6.3V, rlc:CAPACITOR_POL-ALUM-SMT-6.3
- removed D1: Toshiba 1SS416CT, diodes:SCHOTTKYTOSHIBA_CST2
- removed R13: 220, rlc:RESISTOR0603
- removed R16: CTS 741X163102JP, rlc:RESNET_0402_INDIV_X8
- added C4: 0.01uF, rlc:CAPACITOR0603
- added R1, R2: 10K, rlc:RESISTOR0603
- C3: value 0.01uF -> 0.1uF
- C6: value 0.1uF -> 220uF/6.3V; device rlc:CAPACITOR0603 -> rlc:CAPACITOR_POL-ALUM-SMT-6.3
- Q1: value SI2302CDS -> 2N7002; device transistor-fet:SOT23_SI2302 -> transistor-fet:SOT23_2N7002
- R4: value 160K -> NS
- R8: value 10K -> 220
- R9: value NS -> CTS 741X163102JP; device rlc:RESISTOR0603 -> rlc:RESNET_0402_INDIV_X8
- renumbered R10 to R5, R11 to R6, R12 to R7
Connections:
- removed net VCC_AVR: C1.1, C3.1, C7.P, D1.K, R8.2, U1.AVCC, U1.VCC@4, U1.VCC@6
- net D3: now also R8.1; no longer R13.1
- net GND: now also C4.2, C6.N, SV1.3, SV2.3, SV3.3; no longer C6.2, C7.N, R4.1
- net LED_R: now also R8.2; no longer R13.2
- net MOSI: now also R9E.1; no longer R16E.1
- net N$10: now also Q1.D, R9E.2, R9F.2; no longer R16E.2, SV1.1
- net N$11: now also R9B.1; no longer R16B.1
- net N$12: now also R9A.1; no longer R16A.1
- net N$19: now also R9G.1; no longer R16F.1
- net N$2: now also R9F.1, SV1.1; no longer Q1.D, SV1.3, SV2.3, SV3.3
- net N$20: now also R9H.1; no longer R16G.1
- net N$5: now also R9H.2; no longer R16G.2
- net N$9: now also R9G.2; no longer R16F.2
- net RESET: now also R1.1; no longer R8.1
- net RX: now also R9C.1; no longer R16C.1
- net RXD: now also R9D.2; no longer R16D.2
- net SCL: now also R4.1, R9B.2; no longer R16B.2, R9.1
- net SDA: now also R9A.2; no longer R16A.2
- net SERVO_EN: now also R2.2; no longer R4.2
- net TX: now also R9D.1; no longer R16D.1
- net TXD: now also R9C.2; no longer R16C.2
- net VCC: now also C1.1, C3.1, C4.1, C6.P, R1.2, R2.1, R4.2, U1.AVCC, U1.VCC@4, U1.VCC@6; no longer C6.1, D1.A, R9.2
Other:
- note removed: "470uf"
- moved on the sheet: C3, ISCP, Q1, R4, R8, SV1, SV2, SV3

Commit message: rev-e board
Parts:
- removed I/O: (no value), con-headers:MA04-1
- removed R4, R5: NS, rlc:RESISTOR0603
- removed R6, R7, R8: 220, rlc:RESISTOR0603
- removed R9: CTS 741X163102JP, rlc:RESNET_0402_INDIV_X8
- added AIN4, AIN5: TEST_POINT_SM_2X2, test-points:TEST_POINT_SM_2X2
- added D1: Toshiba 1SS416CT, diodes:SCHOTTKYTOSHIBA_CST2
- added D13: YEL, led:SMT0603
- added POWER: HDR, M, 3P, con-headers:MA03-1
- added SER_PWR: (no value), con-headers:JMP01VT
- C6: value 220uF/6.3V -> 1000uF/10V; device rlc:CAPACITOR_POL-ALUM-SMT-6.3 -> rlc:CAPACITOR_POLCAP_ALUM_THD_8
- R3: value NS -> CTS 741X163102JP; device rlc:RESISTOR0603 -> rlc:RESNET_0402_INDIV_X8
- renumbered JMP1 to SER_RST, PD2 to D2, PD4 to D4, PD7 to D7
Connections:
- removed net D3: R8.1, U1.PD3
- removed net D5: R7.1, U1.PD5
- removed net D6: R6.1, U1.PD6
- removed net SCL: I/O.1, R4.1, R9B.2
- removed net SDA: I/O.2, R5.1, R9A.2
- new net N$17: D13.A, R3A.2
- new net PWR_IN: C3.1, D1.A, ISCP.2, LEDS.4, POWER.2, SER_PWR.P$1, SV1.2, SV2.2, SV3.2
- net GND: now also D13.C, POWER.3; no longer I/O.4, LEDS.4
- net LED_B: now also U1.PD6; no longer R6.2
- net LED_G: now also U1.PD5; no longer R7.2
- net LED_R: now also U1.PD3; no longer R8.2
- net MOSI: now also R3E.1; no longer R9E.1
- net N$10: now also R3E.2, R3F.2; no longer R9E.2, R9F.2
- net N$11: now also AIN5.P$1; no longer R9B.1
- net N$12: now also AIN4.P$1; no longer R9A.1
- net N$19: now also R3G.1; no longer R9G.1
- net N$2: now also R3F.1; no longer R9F.1
- net N$20: now also R3H.1; no longer R9H.1
- net N$5: now also R3H.2; no longer R9H.2
- net N$9: now also R3G.2; no longer R9G.2
- net RESET: now also POWER.1
- net RX: now also R3C.1; no longer R9C.1
- net RXD: now also R3D.2; no longer R9D.2
- net SCK: now also R3A.1
- net TX: now also R3D.1; no longer R9D.1
- net TXD: now also R3C.2; no longer R9C.2
- net VCC: now also D1.K; no longer C3.1, I/O.3, ISCP.2, R3.1, R4.2, R5.2, SV1.2, SV2.2, SV3.2
- net VCC5: now also SER_PWR.P$2; no longer R3.2
Other:
- note added: "5VDC @ 3A Recommened"
- note added: "6VDC Max Do not exceed 6V!"
- note added: "Write LOW(0) to LED pins to make them turn on."
- note removed: "I2C pull-ups: No stuff for slaves. You only need one set at the master."
- moved on the sheet: CR1, LEDS
