File: hardware/dmx-cat5-board/pcb/serial-receiver.brd (EAGLE design)
At the start: 30 x 20 mm, 12 parts, among them J1 03P_ED1515-ND, J2 03P_ED1515-ND, U3 ST485

Commit message: DMX cat5 board rev-b
Parts:
- removed J4: (no value), con-headers:MA06-1
- removed R4: 4.7K, rlc:0603
- added J3: HDR, FEM, 6P, con-headers:FE06
- added SJ3: SOLDER_JUMPER, rlc:SOLDER_JUMP
- added SRX, STX: SHORT0603, rlc:0603-SHORT
- added TP2, TP6, TP_RE: TEST_POINT_SM_2X2, test-points:TP-SMT-020X020
- C1: value (none) -> 0.1uF
- U3: value ST485 -> SN65176B
- moved SJ2 16.6 mm to (16.9, 15.5), flipped to the bottom, turned to 180 degrees
- moved SJ1 13.4 mm to (15.0, 15.5), flipped to the bottom, turned to 180 degrees
- moved R3 4.88 mm to (6.55, 9.85), turned to 0 degrees
Connections:
- removed net DE: J4.1, R4.2, SJ2.2, U3.3
- new net N$1: J3.2, TP2.1
- new net N$2: J3.6, TP6.1
- new net RX_CONN: J3.4, SJ2.2, SRX.1
- new net TX_CONN: J3.5, SJ3.2, STX.1
- net GND: now also J3.1; no longer J4.6, R4.1
- net RE_: now also TP_RE.1, U3.3; no longer J4.2
- net RX: now also SJ3.1, SRX.2, U3.1; no longer J4.3, U3.4
- net TX: now also SJ2.1, STX.2, U3.4; no longer J4.4, U3.1
- net VCC: now also J3.3; no longer J4.5, SJ2.1
Routing:
- net DE: track 24.1 -> 0.00 mm, vias 2 -> 0
- net VCC: track 30.3 -> 12.4 mm, vias 1 -> 0
- net N$1: track 0.00 -> 16.0 mm
- net N$2: track 0.00 -> 14.7 mm
- net TX_CONN: track 0.00 -> 5.27 mm
- net RX_CONN: track 0.00 -> 5.22 mm
- net TX: track 7.04 -> 12.0 mm
- net RE_: track 24.2 -> 25.3 mm
- net RX: track 9.75 -> 9.87 mm, vias 0 -> 1
Other:
- board text added: "R O B O T A R M Y"
- board text added: "RS-485"
- board text added: "Rev. B"
- board text added: "Transceiver"
- board text removed: "*"
- board text removed: "/|\\"
- board text removed: "RS-485 Transceiver"
- board text removed: "Rev. A"
