File: hardware/dmx-cat5-board/pcb/serial-receiver.sch (EAGLE design)
At the start: 12 parts, among them J1 03P_ED1515-ND, J2 03P_ED1515-ND, U3 ST485

Commit message: DMX cat5 board rev-b
Parts:
- removed J4: (no value), con-headers:MA06-1
- removed R4: 4.7K, rlc:RESISTOR0603
- added J3: HDR, FEM, 6P, con-headers:FE06-1
- added SJ3: SOLDER_JUMPER, rlc:SOLDER_JUMPER
- added SRX, STX: SHORT0603, rlc:SHORT0603
- added TP2, TP6, TP_RE: TEST_POINT_SM_2X2, test-points:TEST_POINT_SM_2X2
- C1: value (none) -> 0.1uF
- U3: value ST485 -> SN65176B
Connections:
- removed net DE: J4.1, R4.2, SJ2.P$2, U3.DE
- new net N$1: J3.2, TP2.P$1
- new net N$2: J3.6, TP6.P$1
- new net RX_CONN: J3.4, SJ2.P$2, SRX.1
- new net TX_CONN: J3.5, SJ3.P$2, STX.1
- net GND: now also J3.1; no longer J4.6, R4.1
- net RE_: now also TP_RE.P$1, U3.DE; no longer J4.2
- net RX: now also SJ3.P$1, SRX.2, U3.R; no longer J4.3, U3.D
- net TX: now also SJ2.P$1, STX.2, U3.D; no longer J4.4, U3.R
- net VCC: now also J3.3; no longer J4.5, SJ2.P$1
Other:
- note added: "Default config is for Receive(slave) mode."
- note added: "For Master(transmit) board cut SRX and STX then bridge SJ1, SJ2 and SJ3."
- note removed: "Default config is for Receive mode."
- moved on the sheet: C1, J1, J2, R1, R2, R3, SJ1, SJ2
